File: 3.3V 2A output stage.kicad_sch (KiCad schematic)
At the start: 61 parts, among them U201 MP1584EN, U202 LT3045xMSE, U203 LT3045xMSE, U204 LT3045xMSE, U205 LT3045xMSE

Commit message: project structing
Changed lines of the file:
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@@
 		)
 	)
-	(global_label "ENABLE"
-		(shape bidirectional)
+	(hierarchical_label "ENABLE"
+		(shape input)
 		(at 41.91 62.23 180)
-		(fields_autoplaced yes)
 		(effects
 			(font
@@
 			(justify right)
 		)
-		(property "Intersheetrefs" "${INTERSHEET_REFS}"
-			(at 30.7983 62.23 0)
-			(effects
-				(font
-					(size 1.27 1.27)
-				)
-				(justify right)
-				(hide yes)
-			)
-		)
 	)
