File: Low noise power supply.kicad_sch (KiCad schematic)
At the start: 113 parts, among them K1 RZ03-1A4-D012, Q1 BC817, Q2 BC807, Q3 BC817, U1 LT3045xMSE, U2 LT3045xMSE, U3 LM317T, U4 78L05, U5 MP1584EN

Commit message: new power stage output 3V3 2A
Other:
- added sheet 3.3V 2A output stage (3.3V 2A output stage.kicad_sch)
- moved on the sheet: C62, R22, R23
Changed lines of the file:
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@@
 	)
 	(junction
-		(at 139.7 74.93)
+		(at 138.43 76.2)
 		(diameter 0)
 		(color 0 0 0 0)
@@
 	)
 	(junction
-		(at 101.6 74.93)
+		(at 100.33 76.2)
 		(diameter 0)
 		(color 0 0 0 0)
@@
 	(wire
 		(pts
-			(xy 124.46 67.31) (xy 139.7 67.31)
+			(xy 123.19 68.58) (xy 138.43 68.58)
 		)
 		(stroke
@@
 	(wire
 		(pts
-			(xy 101.6 74.93) (xy 107.95 74.93)
+			(xy 100.33 76.2) (xy 106.68 76.2)
 		)
 		(stroke
@@
 	(wire
 		(pts
-			(xy 101.6 67.31) (xy 101.6 74.93)
+			(xy 100.33 68.58) (xy 100.33 76.2)
 		)
 		(stroke
@@
 	(wire
 		(pts
-			(xy 27.94 181.61) (xy 40.64 181.61)
+			(xy 36.83 181.61) (xy 40.64 181.61)
 		)
 		(stroke
@@
 	(wire
 		(pts
-			(xy 133.35 74.93) (xy 139.7 74.93)
+			(xy 132.08 76.2) (xy 138.43 76.2)
 		)
 		(stroke
@@
 	(wire
 		(pts
-			(xy 116.84 67.31) (xy 101.6 67.31)
+			(xy 115.57 68.58) (xy 100.33 68.58)
 		)
 		(stroke
@@
 	(wire
 		(pts
-			(xy 139.7 67.31) (xy 139.7 74.93)
+			(xy 138.43 68.58) (xy 138.43 76.2)
 		)
 		(stroke
@@
 	(wire
 		(pts
-			(xy 115.57 74.93) (xy 125.73 74.93)
+			(xy 114.3 76.2) (xy 124.46 76.2)
 		)
 		(stroke
@@
 	(wire
 		(pts
-			(xy 101.6 74.93) (xy 101.6 76.2)
+			(xy 100.33 76.2) (xy 100.33 77.47)
 		)
 		(stroke
@@
 	(wire
 		(pts
-			(xy 171.45 34.29) (xy 180.34 34.29)
+			(xy 176.53 34.29) (xy 180.34 34.29)
 		)
 		(stroke
@@
 	(wire
 		(pts
-			(xy 139.7 74.93) (xy 139.7 76.2)
+			(xy 138.43 76.2) (xy 138.43 77.47)
 		)
 		(stroke
@@
 	(wire
 		(pts
-			(xy 229.87 134.62) (xy 250.19 134.62)
+			(xy 238.76 134.62) (xy 250.19 134.62)
 		)
 		(stroke
@@
 		)
 	)
-	(label "ENABLE"
-		(at 171.45 34.29 0)
+	(global_label "ENABLE"
+		(shape bidirectional)
+		(at 238.76 134.62 180)
+		(fields_autoplaced yes)
 		(effects
 			(font
 				(size 1.27 1.27)
 			)
-			(justify left bottom)
+			(justify right)
+		)
+		(property "Intersheetrefs" "${INTERSHEET_REFS}"
+			(at 227.6483 134.62 0)
+			(effects
+				(font
+					(size 1.27 1.27)
+				)
+				(justify right)
+				(hide yes)
+			)
 		)
 	)
-	(label "ENABLE"
-		(at 229.87 134.62 0)
+	(global_label "ENABLE"
+		(shape bidirectional)
+		(at 176.53 34.29 180)
+		(fields_autoplaced yes)
 		(effects
 			(font
 				(size 1.27 1.27)
 			)
-			(justify left bottom)
+			(justify right)
+		)
+		(property "Intersheetrefs" "${INTERSHEET_REFS}"
+			(at 165.4183 34.29 0)
+			(effects
+				(font
+					(size 1.27 1.27)
+				)
+				(justify right)
+				(hide yes)
+			)
 		)
 	)
-	(label "ENABLE"
-		(at 27.94 181.61 0)
+	(global_label "ENABLE"
+		(shape bidirectional)
+		(at 36.83 181.61 180)
+		(fields_autoplaced yes)
 		(effects
 			(font
 				(size 1.27 1.27)
 			)
-			(justify left bottom)
+			(justify right)
+		)
+		(property "Intersheetrefs" "${INTERSHEET_REFS}"
+			(at 25.7183 181.61 0)
+			(effects
+				(font
+					(size 1.27 1.27)
+				)
+				(justify right)
+				(hide yes)
+			)
+		)
+	)
+	(hierarchical_label "+15V"
+		(shape output)
+		(at 154.94 207.01 0)
+		(effects
+			(font
+				(size 1.27 1.27)
+			)
+			(justify left)
 		)
 	)
@@
 	(symbol
 		(lib_id "Device:C")
-		(at 120.65 67.31 90)
+		(at 119.38 68.58 90)
 		(unit 1)
 		(exclude_from_sim no)
@@
 		(fields_autoplaced yes)
 		(property "Reference" "C62"
-			(at 120.65 59.69 90)
+			(at 119.38 60.96 90)
 			(effects
 				(font
@@
 		)
 		(property "Value" "2n2"
-			(at 120.65 62.23 90)
+			(at 119.38 63.5 90)
 			(effects
 				(font
@@
 		)
 		(property "Footprint" ""
-			(at 124.46 66.3448 0)
+			(at 123.19 67.6148 0)
 			(effects
 				(font
@@
 		)
 		(property "Datasheet" "~"
-			(at 120.65 67.31 0)
+			(at 119.38 68.58 0)
 			(effects
 				(font
@@
 		)
 		(property "Description" "Unpolarized ceramic capacitor"
-			(at 120.65 67.31 0)
+			(at 119.38 68.58 0)
 			(effects
 				(font
@@
 		)
 		(property "MPN" "CC1206KKX7RZBB222"
-			(at 120.65 67.31 0)
+			(at 119.38 68.58 0)
 			(effects
 				(font
@@
 	(symbol
 		(lib_id "power:Earth")
-		(at 139.7 76.2 0)
+		(at 138.43 77.47 0)
 		(unit 1)
 		(exclude_from_sim no)
@@
 		(fields_autoplaced yes)
 		(property "Reference" "#PWR01"
-			(at 139.7 82.55 0)
+			(at 138.43 83.82 0)
 			(effects
 				(font
@@
 		)
 		(property "Value" "GND"
-			(at 139.7 81.28 0)
+			(at 138.43 82.55 0)
 			(effects
 				(font
@@
 		)
 		(property "Footprint" ""
-			(at 139.7 76.2 0)
+			(at 138.43 77.47 0)
 			(effects
 				(font
@@
 		)
 		(property "Datasheet" "~"
-			(at 139.7 76.2 0)
+			(at 138.43 77.47 0)
 			(effects
 				(font
@@
 		)
 		(property "Description" "Power symbol creates a global label with name \"Earth\""
-			(at 139.7 76.2 0)
+			(at 138.43 77.47 0)
 			(effects
 				(font
@@
 	(symbol
 		(lib_id "Device:R")
-		(at 111.76 74.93 90)
+		(at 110.49 76.2 90)
 		(unit 1)
 		(exclude_from_sim no)
@@
 		(dnp no)
 		(property "Reference" "R22"
-			(at 109.474 71.12 90)
+			(at 108.204 72.39 90)
 			(effects
 				(font
@@
 		)
 		(property "Value" "470k"
-			(at 114.3 71.12 90)
+			(at 113.03 72.39 90)
 			(effects
 				(font
@@
 		)
 		(property "Footprint" ""
-			(at 111.76 76.708 90)
+			(at 110.49 77.978 90)
 			(effects
 				(font
@@
 		)
 		(property "Datasheet" "~"
-			(at 111.76 74.93 0)
+			(at 110.49 76.2 0)
 			(effects
 				(font
@@
 		)
 		(property "Description" "Resistor"
-			(at 111.76 74.93 0)
+			(at 110.49 76.2 0)
 			(effects
 				(font
@@
 		)
 		(property "MPN" "RC1206FR-07470KL"
-			(at 111.76 74.93 0)
+			(at 110.49 76.2 0)
 			(effects
 				(font
@@
 	(symbol
 		(lib_id "Device:R")
-		(at 129.54 74.93 90)
+		(at 128.27 76.2 90)
 		(unit 1)
 		(exclude_from_sim no)
@@
 		(dnp no)
 		(property "Reference" "R23"
-			(at 127.254 71.12 90)
+			(at 125.984 72.39 90)
 			(effects
 				(font
@@
 		)
 		(property "Value" "470k"
-			(at 132.08 71.12 90)
+			(at 130.81 72.39 90)
 			(effects
 				(font
@@
 		)
 		(property "Footprint" ""
-			(at 129.54 76.708 90)
+			(at 128.27 77.978 90)
 			(effects
 				(font
@@
 		)
 		(property "Datasheet" "~"
-			(at 129.54 74.93 0)
+			(at 128.27 76.2 0)
 			(effects
 				(font
@@
 		)
 		(property "Description" "Resistor"
-			(at 129.54 74.93 0)
+			(at 128.27 76.2 0)
 			(effects
 				(font
@@
 		)
 		(property "MPN" "RC1206FR-07470KL"
-			(at 129.54 74.93 0)
+			(at 128.27 76.2 0)
 			(effects
 				(font
@@
 	(symbol
 		(lib_id "power:GNDPWR")
-		(at 101.6 76.2 0)
+		(at 100.33 77.47 0)
 		(unit 1)
 		(exclude_from_sim no)
@@
 		(fields_autoplaced yes)
 		(property "Reference" "#PWR02"
-			(at 101.6 81.28 0)
+			(at 100.33 82.55 0)
 			(effects
 				(font
@@
 		)
 		(property "Value" "PE"
-			(at 101.473 80.01 0)
+			(at 100.203 81.28 0)
 			(effects
 				(font
@@
 		)
 		(property "Footprint" ""
-			(at 101.6 77.47 0)
+			(at 100.33 78.74 0)
 			(effects
 				(font
@@
 		)
 		(property "Datasheet" ""
-			(at 101.6 77.47 0)
+			(at 100.33 78.74 0)
 			(effects
 				(font
@@
 		)
 		(property "Description" "Power symbol creates a global label with name \"GNDPWR\" , global ground"
-			(at 101.6 76.2 0)
+			(at 100.33 77.47 0)
 			(effects
 				(font
@@
 				)
 			)
+		)
+	)
+	(sheet
+		(at 17.78 271.78)
+		(size 33.02 6.35)
+		(exclude_from_sim no)
+		(in_bom yes)
+		(on_board yes)
+		(dnp no)
+		(stroke
+			(width 0.1524)
+			(type solid)
+		)
+		(fill
+			(color 0 0 0 0.0000)
+		)
+		(property "Sheetname" "3.3V 2A output stage"
+			(at 19.05 274.574 0)
+			(effects
+				(font
+					(size 1.27 1.27)
+				)
+				(justify left bottom)
+			)
+		)
+		(property "Sheetfile" "3.3V 2A output stage.kicad_sch"
+			(at 17.78 278.7146 0)
+			(effects
+				(font
+					(size 1.27 1.27)
+				)
+				(justify left top)
+			)
+		)
+		(instances
+			(project "Low noise power supply"
+				(path "/fca69f12-2166-43a7-ac92-c50992f66d73"
+					(page "2")
+				)
+			)

Commit message: project structing
Parts:
- removed C1, C2, C52: 100n, symbol Device:C
- removed C10, C11, C12, C13, C14, C15, C16, C17, C18, C19, C20, C21, C22, C23, C24, C25, C26, C27, C28, C29, C30, C31, C32, C33, C34, C49, C5, C50, C57, C58, C6, C7, C8, C9: 1000u, symbol Device:C_Polarized
- removed C3, C4: 3300p, symbol Device:C
- removed C35, C41, C47, C48, C53, C56: 100u, symbol Device:C_Polarized
- removed C36, C37, C42, C43, C51, C54, C55: 10u, symbol Device:C
- removed C38, C39, C44, C45: 220u, symbol Device:C_Polarized
- removed C40, C46, C60, C61: 1u, symbol Device:C
- removed C59: 150p, symbol Device:C
- removed C62: 2n2, symbol Device:C
- removed CT1, CT2, CT3, CT4, CT5, CT6: 33u, symbol Device:C_Polarized
- removed D1, D2, D4: 1N4007L, symbol Diode:1N4001
- removed D3: BZV55C12, symbol Diode:BZV55C12
- removed D5: BAT54J, Diode_SMD:D_SOD-323F, symbol Diode:BAT54J
- removed D6: B340, Diode_SMD:D_SMC, symbol Diode:B340
- removed F1: MST-3.15A-250V, symbol Device:Fuse
- removed K1: RZ03-1A4-D012, symbol Relay:G2RL-1A
- removed L1: SQ1515-10uH 4A, symbol Device:L_Ferrite_Coupled
- removed L2, L3: 220u, symbol Device:L_Ferrite
- removed L4: 22u, symbol Device:L_Ferrite
- removed PS1: IRM-60-15, Converter_ACDC:Converter_ACDC_MeanWell_IRM-60-xx_THT, symbol Converter_ACDC:IRM-60-15
- removed Q1, Q3: BC817, Package_TO_SOT_SMD:SOT-23, symbol Transistor_BJT:BC817
- removed Q2: BC807, Package_TO_SOT_SMD:SOT-23, symbol Transistor_BJT:BC807
- removed R1: NTC 10 Ом, symbol Device:R
- removed R10, R8: 0.2, symbol Device:R
- removed R11: 56k2, symbol Device:R
- removed R12, R17: 10k, symbol Device:R
- removed R13: 4k3, symbol Device:R
- removed R14, R6, R7: 240, symbol Device:R
- removed R15: 2k26, symbol Device:R
- removed R16, R9: 20k, symbol Device:R
- removed R18: 180k, symbol Device:R
- removed R19: 300k, symbol Device:R
- removed R2: 750, symbol Device:R
- removed R20: 147k, symbol Device:R
- removed R21: 19k6, symbol Device:R
- removed R22, R23: 470k, symbol Device:R
- removed R3, R4: 47k, symbol Device:R
- removed R5: 2k2, symbol Device:R
- removed RV1: S14K420, symbol Device:Varistor
- removed U1, U2: LT3045xMSE, Package_SO:MSOP-12-1EP_3x4.039mm_P0.65mm_EP1.651x2.845mm, symbol Regulator_Linear:LT3045xMSE
- removed U3: LM317T, Package_TO_SOT_THT:TO-220-3_Vertical, symbol Regulator_Linear:LM317_TO-220
- removed U4: 78L05, Package_TO_SOT_SMD:SOT-23_Handsoldering, symbol Regulator_Linear:L78L05_SOT89
- removed U5: MP1584EN, Package_SO:SOIC-8-1EP_3.9x4.9mm_P1.27mm_EP2.62x3.51mm, symbol Regulator_Switching:MP2303ADN
Connections:
- no-connect marks 2 -> 0
Other:
- sheet 3.3V 2A output stage renamed 3.3V 2A PWM output stage
- added sheet Primary supply (Primary supply.kicad_sch)
- added sheet Universal 1A output stage (Universal 1A output stage.kicad_sch)
- sheet 3.3V 2A PWM output stage ports: added ENABLE; removed none
- note removed: "R8 и R10 выполнить медными проводниками на плате в виде дорожек определенной длины и ширины:"
- note removed: "Вариант 1 - линейный понижающий cтабилизатор"
- note removed: "Вариант 2 - ШИМ понижающий cтабилизатор"
- note removed: "Основная плата"
- note removed: "Плата оконечного каскада стабилизации"
