File: 3.3V 1A PWM output stage.kicad_sch (KiCad schematic)
At the start: 49 parts, among them U206 MP1584EN, U207 LT3045xMSE, U210 LT3045xMSE

Commit message: capacitir add
Parts:
- added C391: 33p, symbol Device:C
- C250: value 150p -> 330p
- R216: value 75k -> 100k
Connections:
- net GND: now also C391.2
- net at C250.1, U206.3 (COMP): now also C391.1
Other:
- moved on the sheet: R217
Changed lines of the file:
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@@
 	)
 	(junction
+		(at 118.11 78.74)
+		(diameter 0)
+		(color 0 0 0 0)
+	)
+	(junction
 		(at 276.86 110.49)
 		(diameter 0)
@@
 	)
 	(junction
-		(at 116.84 66.04)
-		(diameter 0)
-		(color 0 0 0 0)
-	)
-	(junction
 		(at 327.66 110.49)
 		(diameter 0)
@@
 	)
 	(junction
+		(at 121.92 66.04)
+		(diameter 0)
+		(color 0 0 0 0)
+	)
+	(junction
 		(at 375.92 46.99)
 		(diameter 0)
@@
 	)
 	(junction
+		(at 111.76 57.15)
+		(diameter 0)
+		(color 0 0 0 0)
+	)
+	(junction
 		(at 124.46 46.99)
 		(diameter 0)
@@
 	(wire
 		(pts
-			(xy 116.84 66.04) (xy 116.84 68.58)
+			(xy 121.92 66.04) (xy 121.92 68.58)
 		)
 		(stroke
@@
 	(wire
 		(pts
-			(xy 116.84 78.74) (xy 111.76 78.74)
+			(xy 121.92 78.74) (xy 118.11 78.74)
 		)
 		(stroke
@@
 	(wire
 		(pts
+			(xy 121.92 66.04) (xy 125.73 66.04)
+		)
+		(stroke
+			(width 0)
+			(type default)
+		)
+	)
+	(wire
+		(pts
 			(xy 269.24 114.3) (xy 265.43 114.3)
 		)
@@
 	(wire
 		(pts
-			(xy 109.22 52.07) (xy 116.84 52.07)
+			(xy 109.22 52.07) (xy 121.92 52.07)
 		)
 		(stroke
@@
 	(wire
 		(pts
-			(xy 116.84 76.2) (xy 116.84 78.74)
+			(xy 121.92 76.2) (xy 121.92 78.74)
 		)
 		(stroke
@@
 	(wire
 		(pts
+			(xy 118.11 69.85) (xy 118.11 78.74)
+		)
+		(stroke
+			(width 0)
+			(type default)
+		)
+	)
+	(wire
+		(pts
 			(xy 295.91 57.15) (xy 298.45 57.15)
 		)
@@
 	(wire
 		(pts
+			(xy 118.11 78.74) (xy 111.76 78.74)
+		)
+		(stroke
+			(width 0)
+			(type default)
+		)
+	)
+	(wire
+		(pts
 			(xy 295.91 46.99) (xy 295.91 49.53)
 		)
@@
 	(wire
 		(pts
-			(xy 116.84 66.04) (xy 125.73 66.04)
-		)
-		(stroke
-			(width 0)
-			(type default)
-		)
-	)
-	(wire
-		(pts
 			(xy 295.91 52.07) (xy 295.91 49.53)
 		)
@@
 	(wire
 		(pts
+			(xy 118.11 62.23) (xy 118.11 57.15)
+		)
+		(stroke
+			(width 0)
+			(type default)
+		)
+	)
+	(wire
+		(pts
 			(xy 152.4 57.15) (xy 152.4 62.23)
 		)
@@
 	(wire
 		(pts
+			(xy 118.11 57.15) (xy 111.76 57.15)
+		)
+		(stroke
+			(width 0)
+			(type default)
+		)
+	)
+	(wire
+		(pts
 			(xy 353.06 46.99) (xy 350.52 46.99)
 		)
@@
 	(wire
 		(pts
-			(xy 116.84 52.07) (xy 116.84 66.04)
+			(xy 121.92 52.07) (xy 121.92 66.04)
 		)
 		(stroke
@@
 			)
 		)
-		(property "Value" "150p"
+		(property "Value" "330p"
 			(at 107.95 64.7699 0)
 			(show_name no)
@@
 	(symbol
 		(lib_id "Device:R")
-		(at 116.84 72.39 0)
+		(at 121.92 72.39 0)
 		(unit 1)
 		(body_style 1)
@@
 		(in_pos_files yes)
 		(dnp no)
-		(fields_autoplaced yes)
 		(property "Reference" "R217"
-			(at 119.38 71.1199 0)
+			(at 124.714 72.898 0)
 			(show_name no)
 			(do_not_autoplace no)
@@
 		)
 		(property "Value" "40k2"
-			(at 119.38 73.6599 0)
+			(at 124.714 75.438 0)
 			(show_name no)
 			(do_not_autoplace no)
@@
 		)
 		(property "Footprint" ""
-			(at 115.062 72.39 90)
+			(at 120.142 72.39 90)
 			(hide yes)
 			(show_name no)
@@
 		)
 		(property "Datasheet" ""
-			(at 116.84 72.39 0)
+			(at 121.92 72.39 0)
 			(hide yes)
 			(show_name no)
@@
 		)
 		(property "Description" "Resistor"
-			(at 116.84 72.39 0)
+			(at 121.92 72.39 0)
 			(hide yes)
 			(show_name no)
@@
 		)
 		(property "MPN" "RC0805FR-0740K2L"
-			(at 116.84 72.39 0)
+			(at 121.92 72.39 0)
 			(hide yes)
 			(show_name no)
@@
 	)
 	(symbol
+		(lib_id "Device:C")
+		(at 118.11 66.04 0)
+		(mirror y)
+		(unit 1)
+		(body_style 1)
+		(exclude_from_sim no)
+		(in_bom yes)
+		(on_board yes)
+		(in_pos_files yes)
+		(dnp no)
+		(property "Reference" "C391"
+			(at 117.602 68.834 0)
+			(show_name no)
+			(do_not_autoplace no)
+			(effects
+				(font
+					(size 1.27 1.27)
+				)
+				(justify left)
+			)
+		)
+		(property "Value" "33p"
+			(at 117.094 71.882 0)
+			(show_name no)
+			(do_not_autoplace no)
+			(effects
+				(font
+					(size 1.27 1.27)
+				)
+				(justify left)
+			)
+		)
+		(property "Footprint" ""
+			(at 117.1448 69.85 0)
+			(hide yes)
+			(show_name no)
+			(do_not_autoplace no)
+			(effects
+				(font
+					(size 1.27 1.27)
+				)
+			)
+		)
+		(property "Datasheet" ""
+			(at 118.11 66.04 0)
+			(hide yes)
+			(show_name no)
+			(do_not_autoplace no)
+			(effects
+				(font
+					(size 1.27 1.27)
+				)
+			)
+		)
+		(property "Description" "Unpolarized ceramic capacitor"
+			(at 118.11 66.04 0)
+			(hide yes)
+			(show_name no)
+			(do_not_autoplace no)
+			(effects
+				(font
+					(size 1.27 1.27)
+				)
+			)
+		)
+		(property "MPN" "CC0805JRNPO0BN151"
+			(at 118.11 66.04 0)
+			(hide yes)
+			(show_name no)
+			(do_not_autoplace no)
+			(effects
+				(font
+					(size 1.27 1.27)
+				)
+			)
+		)
+		(pin "1"
+		)
+		(pin "2"
+		)
+		(instances
+			(project "Low noise power supply"
+				(path "/fca69f12-2166-43a7-ac92-c50992f66d73/8d320d21-90c8-48af-83c0-ce24a813bc66"
+					(reference "C391")
+					(unit 1)
+				)
+			)
+		)
+	)
+	(symbol
 		(lib_name "C_Polarized_1")
 		(lib_id "Device:C_Polarized")
@@
 			)
 		)
-		(property "Value" "75k"
+		(property "Value" "100k"
 			(at 109.22 73.6599 0)
 			(show_name no)
